File: kicad/vodi.kicad_sch (KiCad schematic)
At the start: 39 parts

Commit message: Updated kicad file
Parts:
- removed R1 (x4), R1.2 (x4), R2.2 (x4): ~, symbol Device:R
- removed R2 (x4): R, symbol Device:R
- added -1, -10, -11, -12, -13, -14, -15, -16, -2, -3, -4, -5, -6, -7, -8, -9, GND1, GND2, GND3, GND4, GND5, GND6, GND7, GND8: ~, symbol Connector:TestPoint
- added R1 (x4), R1.2 (x4), R2.2 (x4): ~, symbol Device:R
- added R2 (x4): R, symbol Device:R
Connections:
- net GND: now also GND1.1, GND2.1, GND3.1, GND4.1, GND5.1, GND6.1, GND7.1, GND8.1, R2.2, R2.2, R2.2, R2.2, R2.2.2, R2.2.2, R2.2.2, R2.2.2
- net U1: now also -11.1, -13.1, -15.1, -2.1, -3.1, -5.1, -7.1, -9.1, R1.1, R1.1, R1.1, R1.1, R1.2.1, R1.2.1, R1.2.1, R1.2.1
- removed net U2: R1.1.2, R1.3.2, R1.4.2, R1.5.2, R10.1, R2.1.1, R2.3.1, R2.4.1, R2.5.1, R3.2, R4.1, R5.2, R6.1, R7.2, R8.1, R9.2
- new net: -6.1, R1.4.2, R2.4.1, R7.2, R8.1
- new net: -16.1, R1.2, R1.2.2, R2.1, R2.2.1
- new net: -12.1, R1.2, R1.2.2, R2.1, R2.2.1
- new net: -14.1, R1.2, R1.2.2, R2.1, R2.2.1
- new net: -4.1, R1.3.2, R2.3.1, R5.2, R6.1
- new net: -10.1, R1.2, R1.2.2, R2.1, R2.2.1
- new net: -8.1, R1.5.2, R10.1, R2.5.1, R9.2
- new net: -1.1, R1.1.2, R2.1.1, R3.2, R4.1
Other:
- note added: "U_{Load}"
- note added: "U_{Shunt}"
